Commit message: set up gazebo

File: description/robot_core.xacro (robot description, xacro)
@@ -46,4 +46,7 @@
         </xacro:inertial_box>
     </link>
+    <gazebo reference='chassis'>
+        <material>Gazebo/White</material>
+    </gazebo>
     <!-- LEFT WHEEL LINK -->
     <joint name='left_wheel_joint' type='continuous'>
@@ -69,4 +72,7 @@
         </xacro:inertial_cylinder>
     </link>
+    <gazebo reference='left_wheel'>
+        <material>Gazebo/Blue</material>
+    </gazebo>
     <!-- RIGHT WHEEL LINK -->
     <joint name='right_wheel_joint' type='continuous'>
@@ -92,4 +98,7 @@
         </xacro:inertial_cylinder>
     </link>
+    <gazebo reference='right_wheel'>
+        <material>Gazebo/Blue</material>
+    </gazebo>
     <!-- CASTER WHEEL LINK -->
     <joint name='caster_wheel_joint' type='fixed'>
@@ -114,3 +123,8 @@
         </xacro:inertial_sphere>
     </link>
+    <gazebo reference='caster_wheel'>
+        <material>Gazebo/Black</material>
+        <mu1 value = '0.0001'/>
+        <mu2 value='0.0001'/>
+    </gazebo>
 </robot>

Commit message: added Lidar on the bot

File: description/robot_core.xacro (robot description, xacro)
@@ -14,4 +14,7 @@
      <material name='black'>
         <color rgba='0 0 0 1' />
+     </material>
+     <material name='red'>
+        <color rgba='1 0 0 1' />
      </material>
      <!-- BASE LINK -->
