Commit message: added ros2_control configs

File: description/lidar.xacro (robot description, xacro)
@@ -25,5 +25,5 @@
         <sensor name='laser' type='ray'>
             <pose> 0 0 0 0 0 0</pose>
-            <visualize>false</visualize> <!--This is to turn lasers on/off(true/false) in Gazebo-->
+            <visualize>false</visualize> <!--This is to turn lasers on/off(true/false  ) in Gazebo-->
             <update_rate>10</update_rate>
             <ray>
@@ -44,5 +44,5 @@
             <plugin name='laser_controller' filename='libgazebo_ros_ray_sensor.so'>
                 <ros>
-                    <argument>~/out:=scan</argument>
+                <argument>--ros-args --remap ~/out:=scan</argument>
                 </ros>
                 <output_type>sensor_msgs/LaserScan</output_type>

File: description/robot.urdf.xacro (robot description, xacro)
@@ -2,7 +2,8 @@
 <robot xmlns:xacro="http://www.ros.org/wiki/xacro"  name="robot">
     <xacro:include filename="robot_core.xacro"/>
-    <xacro:include filename="gazebo_control.xacro"/>
+    <!-- <xacro:include filename="gazebo_control.xacro"/> -->
+    <xacro:include filename="ros2_control.xacro"/>
     <xacro:include filename="lidar.xacro"/>
+    <xacro:include filename="depth_camera.xacro"/>
     <!-- <xacro:include filename="camera.xacro"/> -->
-    <xacro:include filename="depth_camera.xacro"/>
 </robot>

File: description/robot_core.xacro (robot description, xacro)
@@ -68,5 +68,5 @@
         <collision>
             <geometry>
-                <cylinder radius='0.05' length='0.04'/>
+                <sphere radius='0.05'/>
             </geometry>
         </collision>
@@ -94,5 +94,5 @@
         <collision>
             <geometry>
-                <cylinder radius='0.05' length='0.04'/>
+                <sphere radius='0.05'/>
             </geometry>
         </collision>
